Commit message: Add collision and inertial to UGV URDF. Also uptade TR NOTE

File: ugv-project/src/ugv_description/urdf/ugv.urdf (robot description, URDF)
Before this commit: robot ugv, 5 links, 4 joints
Links:
- link base_link: mass None -> 5.0
- link left_back_wheel: mass None -> 0.5
- link left_front_wheel: mass None -> 0.5
- link right_back_wheel: mass None -> 0.5
- link right_front_wheel: mass None -> 0.5

Commit message: Add lidar to UGV and add details about Lidar in Turkish Note

File: ugv-project/src/ugv_description/urdf/ugv.urdf (robot description, URDF)
Before this commit: robot ugv, 5 links, 4 joints
Links:
- added link lidar_link, mass 0.1; collision cylinder length=0.05 radius=0.04; visual cylinder length=0.05 radius=0.04
Joints:
- added joint lidar_joint: type fixed, parent base_link, child lidar_link, origin xyz=0.1 0 0.245 rpy=0 0 0
